File: Folder_Structure/Projects/Client Name/Project Name - Copy/Design/rev01/rev01_1/DesingCourse_Project/DesingCourse_Project.kicad_sch (KiCad schematic)
At the start: 0 parts

Commit message: Update 2
KiCAD project creation
Schematica flat hierarqchy with block diagram
Other:
- removed sheet BLOCK_DIAGRAM
- removed sheet CAN
- removed sheet FILTERS
- removed sheet MCU
- removed sheet MECHANICAL
- removed sheet MOSFET
- removed sheet MOSFET_DRIVER
- removed sheet OVERVIEW
- note removed: "ESC_Rev01_1"
- title: ESC_rev01_1 -> Example project
