File: Folder_Structure/Projects/Client Name/Project Name/Design/rev01/rev01_1/DesingCourse_Project/MOSFET_DRIVER.kicad_sch (KiCad schematic)
At the start: 0 parts

Commit message: Update 4
Finish the MOSFET DRIVE page
Parts:
- added C18, C19, C20, C39, C40, C41: 100n, symbol Device:C
- added C21, C29, C30, C31, C32: 2u2, symbol Device:C
- added C22, C23, C24, C25, C26, C27, C35: 1u, symbol Device:C
- added C28: 22n, symbol Device:C
- added C33: 10n, symbol Device:C
- added C34: 120p, symbol Device:C
- added C36, C37, C38: 10u, symbol Device:C
- added D4: PMEG6020AELR, Diode_SMD:Nexperia_CFP3_SOD-123W, symbol Diode:PMEG6020AELR
- added D5: BAT60A, Diode_SMD:D_SOD-323, symbol Diode:BAT60A
- added L1: 22u, symbol Device:L
- added NT1: NetTie_2, symbol Device:NetTie_2
- added R11, R14: 10k, symbol Device:R
- added R12: 16k, symbol Device:R
- added R13: 205k, symbol Device:R
- added R15: 1M, symbol Device:R
- added R16: 18K, symbol Device:R
- added R17: 3K3, symbol Device:R
- added R18, R20, R22: 39k, symbol Device:R
- added R19, R21, R23: 2k2, symbol Device:R
- added U2: DRV8302DCA, DCA56_6P35X3P61, symbol DRV8302DCA:DRV8302DCA
Connections:
- new net: C21.1, U2.27 (AVDD)
- new net: C33.1, R12.1
- new net +VDC: C18.1, C19.1, C20.1, C22.1, C23.1, C24.1, C25.1, C26.1, C27.1, U2.29 (PVDD1), U2.53 (PVDD2), U2.54 (PVDD2)
- new net BIAS: R15.1, U2.49 (BIAS)
- new net BR_SO1: U2.25 (SO1)
- new net BR_SO2: U2.26 (SO2)
- new net BST_1: C41.1, U2.48 (BST_A)
- new net BST_2: C40.1, U2.43 (BST_B)
- new net BST_3: C39.1, U2.38 (BST_C)
- new net BST_BK: C35.1, U2.52 (BST_BK)
- new net COMP: C34.1, R12.2, U2.2 (COMP)
- new net CP1: C28.1, U2.14 (CP1)
- new net CP2: C28.2, U2.15 (CP2)
- new net DC_CAL: U2.12 (DC_CAL)
- new net DTC: R11.2, U2.7 (DTC)
- new net DVDD: NT1.1, U2.23 (DVDD)
- new net EN_GATE: U2.16 (EN_GATE)
- new net FAULT: R14.2, U2.6 (nFAULT)
- new net GND: C18.2, C19.2, C20.2, C21.2, C22.2, C23.2, C24.2, C25.2, C26.2, C27.2, C29.2, C30.2, C31.2, C32.2, C33.2, C34.2, C36.2, C37.2, C38.2, D4.2 (A), R11.1, R13.1, R15.2, R17.2, R19.2, R21.2, R23.2, U2.10 (GAIN), U2.28 (AGND), U2.57 (EPAD), U2.8 (M_PWM)
- new net GVDD: C29.1, C30.1, U2.13 (GVDD)
- new net H1: U2.17 (INH_A)
- new net H1_LOW: U2.44 (SL_A)
- new net H1_VS: C41.2, R18.1, U2.46 (SH_A)
- new net H2: U2.19 (INH_B)
- new net H2_LOW: U2.39 (SL_B)
- new net H2_VS: C40.2, R20.1, U2.41 (SH_B)
- new net H3: U2.21 (INH_C)
- new net H3_LOW: U2.34 (SL_C)
- new net H3_VS: C39.2, R22.1, U2.36 (SH_C)
- new net L1: U2.18 (INL_A)
- new net L2: U2.20 (INL_B)
- new net L3: U2.22 (INL_C)
- new net M_H1: U2.47 (GH_A)
- new net M_H2: U2.42 (GH_B)
- new net M_H3: U2.37 (GH_C)
- new net M_L1: U2.45 (GL_A)
- new net M_L2: U2.40 (GL_B)
- new net M_L3: U2.35 (GL_C)
- new net OC_ADJ: C31.1, C32.1, NT1.2, U2.11 (OC_ADJ)
- new net P3V3: R14.1, U2.24 (REF), U2.9 (M_OC)
- new net P5V: D5.1 (K)
- new net P5V_DRV: C36.1, C37.1, C38.1, D5.2 (A), L1.2, R16.1
- new net PH: C35.2, D4.1 (K), L1.1, U2.50 (PH), U2.51 (PH)
- new net RT_CLK: R13.2, U2.1 (RT_CLK)
- new net S1_N: U2.33 (SN1)
- new net S1_P: U2.30 (SP2), U2.32 (SP1)
- new net S2_N: U2.31 (SN2)
- new net SENS1: R18.2, R19.1
- new net SENS2: R20.2, R21.1
- new net SENS3: R22.2, R23.1
- new net VSENSE: R16.2, R17.1, U2.3 (VSENSE)
- no-connect marks 0 -> 4
Other:
- note added: "1uF DECOUPLING CAPS PLACE AS CLOSE AS POSSIBLE TO THE IC"
- note added: "BOOTSTRAP CAPs"
- note added: "BULK CAPACTIANCE KEEPAS CLOSE AS POSSIBLE TOTHE IC AND HE DRIVER INPUT LOOP"
- note added: "H#_VS"
- note added: "INPUT"
- note added: "MCU SENSING FEEDBACK FRO EACH PHASE"
- note added: "MOSFER DRIVER"
- note added: "OUTPORTS"
- note added: "PHASE 1"
- note added: "PHASE 2"
- note added: "PHASE 3"
- note added: "SENSE 1 - PHASE 1"
- note added: "SENSE 2 - PHASE 2"
- note added: "VSENSE KEEP AWAY FROM NOISY TRACKS AND COMPONENTS"
