File: Folder_Structure/Projects/Client Name/Project Name/Design/rev01/rev01_1/DesingCourse_Project/MOSFET_DRIVER.kicad_sch (KiCad schematic)
At the start: 42 parts, among them U4 DRV8302DCA

Commit message: Update18
Layout finished, clean up or layout and designators.
Connections:
- net Node9: now reaches C31.1, U4.27 (AVDD)
Changed lines of the file:
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@@
 	(wire
 		(pts
+			(xy 88.9 116.84) (xy 100.33 116.84)
+		)
+		(stroke
+			(width 0)
+			(type default)
+		)
+	)
+	(wire
+		(pts
 			(xy 256.54 106.68) (xy 256.54 109.22)
 		)
@@
 	(wire
 		(pts
-			(xy 100.33 116.84) (xy 88.9 116.84)
-		)
-		(stroke
-			(width 0)
-			(type default)
-		)
-	)
-	(wire
-		(pts
 			(xy 153.67 142.24) (xy 160.02 142.24)
 		)
@@
 		)
 	)
-	(label ""
-		(at 90.17 116.84 0)
-		(effects
-			(font
-				(size 1.27 1.27)
-			)
-			(justify left bottom)
-		)
-	)
 	(label "H2_VS"
 		(at 256.54 109.22 0)
@@
 			)
 		)
-		(property "Description" "RES 18k OHM 0603 ±1% 1/10W"
+		(property "Description" "Resistor"
 			(at 219.71 68.58 0)
 			(effects
@@
 			)
 		)
-		(property "Description" "CAP CER 2.2UF 6.3V X5R 0603"
+		(property "Description" "Unpolarized capacitor"
 			(at 55.88 81.28 0)
 			(effects
@@
 			)
 		)
-		(property "Description" "RES 10k OHM 0603 ±1% 1/10W"
+		(property "Description" "Resistor"
 			(at 80.01 63.5 0)
 			(effects
@@
 			)
 		)
-		(property "Description" "CAP CER 0.1UF 10V X7R 0603"
+		(property "Description" "Unpolarized capacitor"
 			(at 168.91 62.23 0)
 			(effects
@@
 			)
 		)
-		(property "Description" "CAP CER 0.1UF 10V X7R 0603"
+		(property "Description" "Unpolarized capacitor"
 			(at 271.78 102.87 0)
 			(effects
@@
 			)
 		)
-		(property "Description" "CAP CER 2.2UF 6.3V X5R 0603"
+		(property "Description" "Unpolarized capacitor"
 			(at 62.23 100.33 0)
 			(effects
@@
 			)
 		)
-		(property "Description" "CAP CER 10nF 50V X7R 0603"
+		(property "Description" "Unpolarized capacitor"
 			(at 50.8 59.69 0)
 			(effects
@@
 			)
 		)
-		(property "Description" "RES 2k2 OHM 0603 ±1% 1/10W"
+		(property "Description" "Resistor"
 			(at 240.03 149.86 0)
 			(effects
@@
 			)
 		)
-		(property "Description" "CAP CER 0.1UF 10V X7R 0603"
+		(property "Description" "Unpolarized capacitor"
 			(at 166.37 135.89 0)
 			(effects
@@
 			)
 		)
-		(property "Description" "RES 3k3 OHM 0603 ±1% 1/10W"
+		(property "Description" "Resistor"
 			(at 219.71 78.74 0)
 			(effects
@@
 			)
 		)
-		(property "Description" "RES 1M OHM 0603 ±1% 1/10W"
+		(property "Description" "Resistor"
 			(at 168.91 73.66 0)
 			(effects
@@
 			)
 		)
-		(property "Description" "CAP CER 22nF 100V X7R 0603"
+		(property "Description" "Unpolarized capacitor"
 			(at 78.74 87.63 0)
 			(effects
@@
 			)
 		)
-		(property "Description" "CAP CER 1UF 100V X7R 0603"
+		(property "Description" "Unpolarized capacitor"
 			(at 184.15 41.91 0)
 			(effects
@@
 			)
 		)
-		(property "Description" "CAP CER 0.1UF 10V X7R 0603"
+		(property "Description" "Unpolarized capacitor"
 			(at 256.54 102.87 0)
 			(effects
@@
 			)
 		)
-		(property "Description" "CAP CER 2.2UF 6.3V X5R 0603"
+		(property "Description" "Unpolarized capacitor"
 			(at 55.88 100.33 0)
 			(effects
@@
 			)
 		)
-		(property "Description" "CAP CER 10UF 16V X5R 1210"
+		(property "Description" "Unpolarized capacitor"
 			(at 204.47 67.31 0)
 			(effects
@@
 			)
 		)
-		(property "Description" "CAP CER 0.1UF 10V X7R 0603"
+		(property "Description" "Unpolarized capacitor"
 			(at 160.02 135.89 0)
 			(effects
@@
 			)
 		)
-		(property "Description" "RES 205k OHM 0603 ±1% 1/10W"
+		(property "Description" "Resistor"
 			(at 78.74 50.8 0)
 			(effects
@@
 			)
 		)
-		(property "Description" "RES 10k OHM 0603 ±1% 1/10W"
+		(property "Description" "Resistor"
 			(at 80.01 66.04 0)
 			(effects
@@
 			)
 		)
-		(property "Description" "RES 39k OHM 0603 ±1% 1/10W"
+		(property "Description" "Resistor"
 			(at 270.51 139.7 0)
 			(effects
@@
 			)
 		)
-		(property "Description" "CAP CER 2.2UF 6.3V X5R 0603"
+		(property "Description" "Unpolarized capacitor"
 			(at 88.9 121.92 0)
 			(effects
@@
 			)
 		)
-		(property "Description" "CAP CER 1UF 100V X7R 0603"
+		(property "Description" "Unpolarized capacitor"
 			(at 189.23 41.91 0)
 			(effects
@@
 			)
 		)
-		(property "Description" "CAP CER 10UF 16V X5R 1210"
+		(property "Description" "Unpolarized capacitor"
 			(at 210.82 67.31 0)
 			(effects
@@
 			)
 		)
-		(property "Description" "RES 2k2 OHM 0603 ±1% 1/10W"
+		(property "Description" "Resistor"
 			(at 255.27 149.86 0)
 			(effects
@@
 			)
 		)
-		(property "Description" "CAP CER 1UF 100V X7R 0603"
+		(property "Description" "Unpolarized capacitor"
 			(at 209.55 41.91 0)
 			(effects
@@
 			)
 		)
-		(property "Description" "CAP CER 1UF 100V X7R 0603"
+		(property "Description" "Unpolarized capacitor"
 			(at 194.31 41.91 0)
 			(effects
@@
 			)
 		)
-		(property "Description" "CAP CER 2.2UF 6.3V X5R 0603"
+		(property "Description" "Unpolarized capacitor"
 			(at 62.23 81.28 0)
 			(effects
@@
 			)
 		)
-		(property "Description" "CAP CER 120pF 50V X7R 0603"
+		(property "Description" "Unpolarized capacitor"
 			(at 60.96 59.69 0)
 			(effects
@@
 			)
 		)
-		(property "Description" "CAP CER 10UF 16V X5R 1210"
+		(property "Description" "Unpolarized capacitor"
 			(at 198.12 67.31 0)
 			(effects
@@
 			)
 		)
-		(property "Description" "CAP CER 1UF 100V X7R 0603"
+		(property "Description" "Unpolarized capacitor"
 			(at 199.39 41.91 0)
 			(effects
@@
 			)
 		)
-		(property "Description" "RES 2k2 OHM 0603 ±1% 1/10W"
+		(property "Description" "Resistor"
 			(at 270.51 149.86 0)
 			(effects
@@
 			)
 		)
-		(property "Description" "CAP CER 0.1UF 10V X7R 0603"
+		(property "Description" "Unpolarized capacitor"
 			(at 241.3 102.87 0)
 			(effects
@@
 			)
 		)
-		(property "Description" "CAP CER 1UF 100V X7R 0603"
+		(property "Description" "Unpolarized capacitor"
 			(at 204.47 41.91 0)
 			(effects
@@
 			)
 		)
-		(property "Description" "RES 16k OHM 0603 ±1% 1/10W"
+		(property "Description" "Resistor"
 			(at 55.88 53.34 0)
 			(effects
@@
 			)
 		)
-		(property "Description" "RES 39k OHM 0603 ±1% 1/10W"
+		(property "Description" "Resistor"
 			(at 255.27 139.7 0)
 			(effects
@@
 			)
 		)
-		(property "Description" "CAP CER 0.1UF 10V X7R 0603"
+		(property "Description" "Unpolarized capacitor"
 			(at 153.67 135.89 0)
 			(effects
@@
 			)
 		)
-		(property "Description" "RES 39k OHM 0603 ±1% 1/10W"
+		(property "Description" "Resistor"
 			(at 240.03 139.7 0)
 			(effects
