File: Folder_Structure/Projects/Client Name/Project Name/Design/rev01/rev01_1/DesingCourse_Project/OVERVIEW.kicad_sch (KiCad schematic)
At the start: 0 parts

Commit message: Update 6
SCH and LIB for MOSFET page done, missing passive components
Other:
- company: (none) -> Integro Consulting AB
- title: (none) -> PCB Mastery Project
Changed lines of the file:
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@@
 	(generator_version "9.0")
 	(paper "A4")
+	(title_block
+		(title "PCB Mastery Project")
+		(date "2026-01-27")
+		(rev "001")
+		(company "Integro Consulting AB")
+		(comment 1 "TBD")
+		(comment 2 "TBD")
+		(comment 3 "TBD")
+		(comment 4 "Josue Godinez")
+	)
 )
